File: RGBBlinkyCR2032.brd (EAGLE design)
At the start: 33 x 43.2 mm, 13 parts, among them J1 AVR_SPI_PRG_6LABELED

Commit message: 4H foo
Parts:
- removed U$3: USER_HACKABLE, logo:USER_HACKABLE
- added U$4: 4H-LOGO6, 4h:4H_LOGO_6
- R1: value 50 -> 51
- moved S1 0.63 mm to (5.71, 21.6)
Routing:
- net GND: track 112.4 -> 113.0 mm
Other:
- board text added: "18 USC 707"
- board text added: "Cache Makers"
- board text added: "cachemakers.org"
- board text removed: "User Hackable"
Changed lines of the file:
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@@
 <layer number="20" name="Dimension" color="15" fill="1" visible="yes" active="yes"/>
 <layer number="21" name="tPlace" color="7" fill="1" visible="yes" active="yes"/>
-<layer number="22" name="bPlace" color="14" fill="1" visible="yes" active="yes"/>
+<layer number="22" name="bPlace" color="6" fill="1" visible="yes" active="yes"/>
 <layer number="23" name="tOrigins" color="15" fill="1" visible="yes" active="yes"/>
 <layer number="24" name="bOrigins" color="15" fill="1" visible="yes" active="yes"/>
@@
 <hole x="29.21" y="39.37" drill="3.175"/>
 <text x="23.495" y="10.16" size="1.016" layer="21" align="center">1</text>
-<text x="8.255" y="15.24" size="1.016" layer="21" align="center">3</text>
+<text x="8.5725" y="15.24" size="1.016" layer="21" align="center">3</text>
 <text x="9.8425" y="10.16" size="1.016" layer="21" align="center">3</text>
-<text x="16.51" y="23.8125" size="1.016" layer="21" align="center">RGB Blinky</text>
-<text x="6.35" y="25.4" size="1.016" layer="21" align="center">MODE</text>
+<text x="26.9875" y="20.0025" size="1.016" layer="21" align="center">RGB Blinky</text>
+<text x="5.715" y="25.4" size="1.016" layer="21" align="center">MODE</text>
 <text x="16.51" y="8.89" size="1.016" layer="22" rot="MR0" align="center">User Hackable
 RGB Blinky</text>
@@
 <text x="5.08" y="8.255" size="1.27" layer="21" align="center">+</text>
 <text x="2.54" y="8.255" size="1.27" layer="21" align="center">-</text>
-<text x="16.8275" y="25.0825" size="1.016" layer="21" align="bottom-center">User Hackable</text>
+<text x="16.8275" y="24.13" size="1.016" layer="21" align="bottom-center">Cache Makers</text>
+<text x="23.1775" y="28.8925" size="0.6096" layer="21" rot="R50" align="center">18 USC 707</text>
+<text x="16.8275" y="23.1775" size="0.8128" layer="21" align="bottom-center">cachemakers.org</text>
 </plain>
 <attributes>
@@
 <attribute name="VALUE" x="13.0429" y="2.0066" size="1.27" layer="27" ratio="10"/>
 </element>
-<element name="R1" library="SparkFun-Resistors" package="AXIAL-0.3" value="50" x="16.51" y="11.43" smashed="yes" rot="R180">
+<element name="R1" library="SparkFun-Resistors" package="AXIAL-0.3" value="51" x="16.51" y="11.43" smashed="yes" rot="R180">
 <attribute name="VALUE" x="14.2875" y="11.43" size="1.016" layer="21" font="vector" ratio="15" rot="R180" align="center-right"/>
 </element>
-<element name="S1" library="barbary_enterprises" package="TACTILE-PTH" value="" x="6.35" y="21.59" smashed="yes"/>
+<element name="S1" library="barbary_enterprises" package="TACTILE-PTH" value="" x="5.715" y="21.59" smashed="yes"/>
 <element name="U$1" library="SparkFun-DigitalIC" package="DIP08" value="TINY85" x="16.51" y="17.78" smashed="yes" rot="R270">
 <attribute name="VALUE" x="15.875" y="20.955" size="1.27" layer="27" ratio="10" rot="R270"/>
@@
 <attribute name="VALUE" x="20.828" y="27.94" size="1.6764" layer="28" font="vector" rot="MR0"/>
 </element>
-<element name="U$3" library="logo" package="USER_HACKABLE" value="USER_HACKABLE" x="16.51" y="34.29"/>
-<element name="SG1" library="SparkFun-Electromechanical" package="BUZZER-12MM" value="BUZZER" x="27.305" y="13.0175" smashed="yes">
-<attribute name="NAME" x="26.67" y="12.7" size="0.6096" layer="25" ratio="10"/>
-<attribute name="VALUE" x="22.733" y="11.43" size="0.6096" layer="27" ratio="10" rot="R90"/>
-</element>
+<element name="SG1" library="SparkFun-Electromechanical" package="BUZZER-12MM" value="BUZZER" x="27.305" y="13.0175" smashed="yes"/>
 <element name="R2" library="SparkFun-Sensors" package="PHOTOCELL" value="PHOTOCELL" x="5.08" y="13.97" smashed="yes" rot="R180">
-<attribute name="VALUE" x="5.08" y="16.1925" size="0.8128" layer="27" align="bottom-center"/>
+<attribute name="VALUE" x="5.08" y="16.51" size="0.8128" layer="27" align="bottom-center"/>
 </element>
 <element name="JP1" library="SparkFun-Connectors" package="1X03" value="" x="2.54" y="10.16" smashed="yes">
@@
 <attribute name="VALUE" x="31.75" y="13.335" size="1.27" layer="27" rot="R180"/>
 </element>
+<element name="U$4" library="4h" package="4H_LOGO_6" value="4H-LOGO6" x="16.51" y="33.655"/>
 </elements>
 <signals>
@@
 <contactref element="S1" pad="3"/>
 <contactref element="J1" pad="5"/>
-<wire x1="3.0988" y1="19.3294" x2="9.6012" y2="19.3294" width="0.8128" layer="16"/>
-<wire x1="9.6012" y1="19.3294" x2="11.8618" y2="21.59" width="0.8128" layer="16"/>
+<wire x1="2.4638" y1="19.3294" x2="8.9662" y2="19.3294" width="0.8128" layer="16"/>
+<wire x1="8.9662" y1="19.3294" x2="11.8618" y2="21.59" width="0.8128" layer="16"/>
 <wire x1="11.8618" y1="21.59" x2="12.7" y2="21.59" width="0.8128" layer="16"/>
 <wire x1="30.48" y1="27.305" x2="30.1625" y2="27.305" width="0.3048" layer="1"/>
@@
 <wire x1="27.94" y1="27.305" x2="23.495" y2="27.305" width="0.8128" layer="16"/>
 <wire x1="23.495" y1="27.305" x2="16.51" y2="34.29" width="0.8128" layer="16"/>
-<wire x1="9.6012" y1="23.8506" x2="10.16" y2="24.13" width="0.8128" layer="16"/>
+<wire x1="8.9662" y1="23.8506" x2="10.16" y2="24.13" width="0.8128" layer="16"/>
 <wire x1="10.16" y1="24.13" x2="15.24" y2="24.13" width="0.8128" layer="16"/>
 <wire x1="15.24" y1="24.13" x2="15.24" y2="13.97" width="0.8128" layer="16"/>
@@
 <wire x1="15.24" y1="24.13" x2="15.24" y2="33.02" width="0.8128" layer="16"/>
 <wire x1="15.24" y1="33.02" x2="16.51" y2="34.29" width="0.8128" layer="16"/>
-<wire x1="3.0988" y1="23.8506" x2="9.6012" y2="23.8506" width="0.8128" layer="16"/>
+<wire x1="2.4638" y1="23.8506" x2="8.9662" y2="23.8506" width="0.8128" layer="16"/>
 <contactref element="SG1" pad="+"/>
 <contactref element="R2" pad="2"/>

Commit message: updating logo
Parts:
- U$4: value 4H-LOGO6 -> (none)
Changed lines of the file:
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@@
 <attribute name="VALUE" x="31.75" y="13.335" size="1.27" layer="27" rot="R180"/>
 </element>
-<element name="U$4" library="4h" package="4H_LOGO_6" value="4H-LOGO6" x="16.51" y="33.655"/>
+<element name="U$4" library="4h" package="4H_LOGO_6" value="" x="16.51" y="33.655"/>
 </elements>
 <signals>
