File: RGBBlinkyCR2032.sch (EAGLE design)
At the start: 13 parts, among them J1 AVR_SPI_PRG_6LABELED

Commit message: 4H foo
Parts:
- removed U$3: USER_HACKABLE, logo:USER_HACKABLE
- added U$4: 4H-LOGO6, 4h:4H-LOGO6
- R1: value 50 -> 51
Changed lines of the file:
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@@
 <part name="U$1" library="SparkFun-DigitalIC" deviceset="ATTINY13" device="DIP" value="TINY85"/>
 <part name="J1" library="barbary_enterprises" deviceset="AVR_SPI_PRG_6" device="LABELED"/>
-<part name="R1" library="SparkFun-Resistors" deviceset="RESISTOR" device="AXIAL-0.3" value="50"/>
+<part name="R1" library="SparkFun-Resistors" deviceset="RESISTOR" device="AXIAL-0.3" value="51"/>
 <part name="RED" library="SparkFun-LED" deviceset="LED" device="5MM"/>
 <part name="GREEN" library="SparkFun-LED" deviceset="LED" device="5MM"/>
@@
 <part name="S1" library="barbary_enterprises" deviceset="TAC_SWITCH" device="PTH"/>
 <part name="U$2" library="battery" deviceset="CR2032" device="THM"/>
-<part name="U$3" library="logo" deviceset="USER_HACKABLE" device=""/>
 <part name="SG1" library="SparkFun-Electromechanical" deviceset="BUZZER" device="PTH" value="BUZZER"/>
 <part name="R2" library="SparkFun-Sensors" deviceset="PHOTOCELL" device="PTH" value="PHOTOCELL"/>
@@
 <part name="SUPPLY3" library="SparkFun-Aesthetics" deviceset="VCC" device=""/>
 <part name="SUPPLY4" library="SparkFun-Aesthetics" deviceset="VCC" device=""/>
+<part name="U$4" library="4h" deviceset="4H-LOGO" device="6"/>
 </parts>
 <sheets>
@@
 <instance part="S1" gate="S" x="40.64" y="15.24"/>
 <instance part="U$2" gate="G$1" x="17.78" y="35.56" rot="R90"/>
-<instance part="U$3" gate="G$1" x="76.2" y="20.32"/>
 <instance part="SG1" gate="G$1" x="83.82" y="40.64" rot="MR0"/>
 <instance part="R2" gate="G$1" x="78.74" y="58.42"/>
@@
 <instance part="SUPPLY3" gate="G$1" x="114.3" y="55.88" rot="R270"/>
 <instance part="SUPPLY4" gate="G$1" x="114.3" y="38.1" rot="R270"/>
+<instance part="U$4" gate="G$1" x="96.52" y="17.78"/>
 </instances>
 <busses>

Commit message: updating logo
Parts:
- U$4: value 4H-LOGO6 -> (none)
